File: Hardware/TJA1050.kicad_sch (KiCad schematic)
At the start: 7 parts, among them J13 Screw_Terminal_01x02, U16 TJA1051T

Commit message: Layout PCB
Parts:
- J13: footprint TerminalBlock:TerminalBlock_bornier-2_P5.08mm -> IVS_FOOTPRINTS:TerminalBlock_bornier-2_P5.08mm
Changed lines of the file:
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@@
     (effects (font (size 1.27 1.27)) (justify right))
   )
-  (hierarchical_label "CAN_RX" (shape input) (at 107.315 69.215 180) (fields_autoplaced)
+  (hierarchical_label "CAN_RX" (shape output) (at 107.315 69.215 180) (fields_autoplaced)
     (effects (font (size 1.27 1.27)) (justify right))
   )
@@
       (effects (font (size 1.27 1.27)) (justify left))
     )
-    (property "Footprint" "TerminalBlock:TerminalBlock_bornier-2_P5.08mm" (at 194.945 66.675 0)
-      (effects (font (size 1.27 1.27)) hide)
-    )
+    (property "Footprint" "IVS_FOOTPRINTS:TerminalBlock_bornier-2_P5.08mm" (at 194.945 66.675 0)
+      (effects (font (size 1.27 1.27)) hide)
+    )

Commit message: Update components
Connections:
- net CANH: now also J13.2 (Pin_2); no longer J13.1 (Pin_1)
- net CANL: now also J13.1 (Pin_1); no longer J13.2 (Pin_2)
Changed lines of the file:
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@@
     )
   )
-  (symbol (lib_id "Connector:Screw_Terminal_01x02") (at 194.945 66.675 0) (unit 1)
-    (in_bom yes) (on_board yes) (dnp no) (fields_autoplaced)
-    (property "Reference" "J13" (at 198.12 66.675 0)
+  (symbol (lib_id "Connector:Screw_Terminal_01x02") (at 194.945 69.215 0) (mirror x) (unit 1)
+    (in_bom yes) (on_board yes) (dnp no)
+    (property "Reference" "J13" (at 198.12 69.215 0)
       (effects (font (size 1.27 1.27)) (justify left))
     )
-    (property "Value" "Screw_Terminal_01x02" (at 198.12 69.215 0)
+    (property "Value" "Screw_Terminal_01x02" (at 198.12 66.675 0)
       (effects (font (size 1.27 1.27)) (justify left))
     )
-    (property "Footprint" "IVS_FOOTPRINTS:TerminalBlock_bornier-2_P5.08mm" (at 194.945 66.675 0)
+    (property "Footprint" "IVS_FOOTPRINTS:TerminalBlock_bornier-2_P5.08mm" (at 194.945 69.215 0)
       (effects (font (size 1.27 1.27)) hide)
     )
-    (property "Datasheet" "~" (at 194.945 66.675 0)
+    (property "Datasheet" "~" (at 194.945 69.215 0)
       (effects (font (size 1.27 1.27)) hide)
     )
