File: Hardware/DriverMotor.kicad_sch (KiCad schematic)
At the start: 4 parts

Commit message: Fix bug schematic
Other:
- sheet MCT8316 ports: added +24V_CS, PA5; removed none
- sheet STM32F103 ports: added PA5; removed none
Changed lines of the file:
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@@
+    (stroke (width 0) (type default))
+  )
+  (wire (pts (xy 112.395 92.075) (xy 127.635 92.075))
     (stroke (width 0) (type default))
   )
@@
   )
   (wire (pts (xy 120.65 80.01) (xy 120.65 77.47))
+    (stroke (width 0) (type default))
+  )
+  (wire (pts (xy 99.06 68.58) (xy 99.06 65.405))
+    (stroke (width 0) (type default))
+  )
+  (wire (pts (xy 99.06 65.405) (xy 142.24 65.405))
     (stroke (width 0) (type default))
   )
@@
       (effects (font (size 1.27 1.27)) (justify left))
     )
+    (pin "PA5" input (at 127.635 92.075 180)
+      (effects (font (size 1.27 1.27)) (justify left))
+    )
     (instances
       (project "DriverMotor"
@@
       (effects (font (size 1.27 1.27)) (justify right))
     )
+    (pin "PA5" output (at 112.395 92.075 0)
+      (effects (font (size 1.27 1.27)) (justify right))
+    )
+    (pin "+24V_CS" input (at 99.06 68.58 90)
+      (effects (font (size 1.27 1.27)) (justify right))
+    )

Commit message: Update README
Changed lines of the file:
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@@
       (effects (font (size 1.27 1.27)) (justify left))
     )
-    (pin "CANRX" output (at 138.43 102.235 270)
+    (pin "CANTX" output (at 138.43 102.235 270)
       (effects (font (size 1.27 1.27)) (justify left))
     )
-    (pin "CANTX" input (at 141.605 102.235 270)
+    (pin "CANRX" input (at 141.605 102.235 270)
       (effects (font (size 1.27 1.27)) (justify left))
     )
