File: Hardware/MCT8316.kicad_sch (KiCad schematic)
At the start: 32 parts, among them J5 Screw_Terminal_01x03, J6 Screw_Terminal_01x03, J7 Conn_01x04_Male, J8 Conn_01x03_Pin, U10 MCT8316, U12 ISO7721DR

Commit message: Update Encoder
Changed lines of the file:
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@@
     (stroke (width 0) (type default))
   )
-  (rectangle (start 18.415 76.835) (end 102.235 186.055)
+  (rectangle (start 18.415 76.835) (end 102.235 142.24)
     (stroke (width 0) (type default))
     (fill (type none))
@@
     (effects (font (size 3 3) (thickness 2) bold) (justify left bottom))
   )
-  (text "Isolation" (at 45.085 184.785 0)
+  (text "Isolation" (at 44.45 137.795 0)
     (effects (font (size 5 5) (thickness 2) bold) (justify left bottom))
   )
