File: Hardware/MCT8316.kicad_sch (KiCad schematic)
At the start: 35 parts, among them J5 Screw_Terminal_01x03, J6 Screw_Terminal_01x03, J7 Conn_01x04_Male, J8 Conn_01x03_Pin, U10 MCT8316, U12 ISO7721DR

Commit message: Complete layout board
Connections:
- net +24V_CS: now also F1.1
- net AVDD: now also U10.27 (AVDD); no longer U10.26 (AVDD)
- net GNDD: now also C22.1, U10.26 (AGND), U10.4 (GND_BK); no longer U10.27 (AGND)
- net MCT.PWM: no longer J7.1 (Pin_1)
- net PWM_BLDC: now also J7.1 (Pin_1)
- net VM: now also F1.2
- net DVDD: now reaches C12.1, U10.1 (DVDD)
Other:
- moved on the sheet: F1
Changed lines of the file:
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@@
   (junction (at 234.95 116.205) (diameter 0) (color 0 0 0 0)
   )
+  (junction (at 147.32 114.3) (diameter 0) (color 0 0 0 0)
+  )
   (junction (at 180.34 186.055) (diameter 0) (color 0 0 0 0)
   )
@@
   )
   (wire (pts (xy 234.95 116.205) (xy 234.95 118.745))
+    (stroke (width 0) (type default))
+  )
+  (wire (pts (xy 145.415 114.3) (xy 147.32 114.3))
     (stroke (width 0) (type default))
   )
@@
     (effects (font (size 1.27 1.27)) (justify left bottom))
   )
-  (label "MCT.PWM" (at 158.75 20.32 180) (fields_autoplaced)
-    (effects (font (size 1.27 1.27)) (justify right bottom))
-  )
   (label "MCT_BRAKE" (at 137.795 136.525 0) (fields_autoplaced)
     (effects (font (size 1.27 1.27)) (justify left bottom))
@@
     (effects (font (size 1.27 1.27)) (justify left bottom))
   )
+  (label "PWM_BLDC" (at 158.75 20.32 180) (fields_autoplaced)
+    (effects (font (size 1.27 1.27)) (justify right bottom))
+  )
   (label "MA" (at 154.305 45.72 0) (fields_autoplaced)
     (effects (font (size 1.27 1.27)) (justify left bottom))
@@
   )
   (label "MCT.FAULT" (at 34.29 217.17 180) (fields_autoplaced)
+    (effects (font (size 1.27 1.27)) (justify right bottom))
+  )
+  (label "DVDD" (at 146.05 120.015 180) (fields_autoplaced)
     (effects (font (size 1.27 1.27)) (justify right bottom))
   )
@@
     )
   )
-  (symbol (lib_id "IVS_SYMBOLS:Fuse") (at 234.95 98.425 180) (unit 1)
+  (symbol (lib_id "IVS_SYMBOLS:Fuse") (at 234.95 98.425 270) (unit 1)
     (in_bom yes) (on_board yes) (dnp no) (fields_autoplaced)
-    (property "Reference" "F1" (at 236.855 97.155 0)
-      (effects (font (size 1.27 1.27)) (justify right))
-    )
-    (property "Value" "30V/3A" (at 236.855 99.695 0)
-      (effects (font (size 1.27 1.27)) (justify right))
-    )
-    (property "Footprint" "Fuse:Fuse_Bourns_MF-RG300" (at 236.728 98.425 90)
+    (property "Reference" "F1" (at 237.49 97.79 90)
+      (effects (font (size 1.27 1.27)) (justify left))
+    )
+    (property "Value" "30V/3A" (at 237.49 100.33 90)
+      (effects (font (size 1.27 1.27)) (justify left))
+    )
+    (property "Footprint" "Fuse:Fuse_Bourns_MF-RG300" (at 234.95 96.647 90)
       (effects (font (size 1.27 1.27)) hide)
     )
@@
         )
       )
+    )
+  )
+  (symbol (lib_id "power:GNDD") (at 145.415 114.3 270) (unit 1)
+    (in_bom yes) (on_board yes) (dnp no) (fields_autoplaced)
+    (property "Reference" "#PWR036" (at 139.065 114.3 0)
+      (effects (font (size 1.27 1.27)) hide)
+    )
+    (property "Value" "GNDD" (at 141.605 114.935 90)
+      (effects (font (size 1.27 1.27)) (justify right))
+    )
+    (property "Footprint" "" (at 145.415 114.3 0)
+      (effects (font (size 1.27 1.27)) hide)
+    )
+    (property "Datasheet" "" (at 145.415 114.3 0)
+      (effects (font (size 1.27 1.27)) hide)
+    )
+    (pin "1")
+    (instances
+      (project "DriverMotor"
+        (path "/8a82bd86-ff43-47ee-a4c0-46ff08914251/719245fa-8c27-4cf8-8d61-6f38548a0446"
+          (reference "#PWR036") (unit 1)
+        )
+      )

Commit message: Update README
Parts:
- added Q2: N_Mosfet, IVS_FOOTPRINTS:SOT23-3, symbol IVS_SYMBOLS:N_Mosfet
- added R36: 1K, IVS_FOOTPRINTS:R_0603, symbol IVS_SYMBOLS:R
Connections:
- net +24V_CS: now also R14.2
- net GND: now also R36.1
- net GNDD: now also C12.1, J8.2 (Pin_2)
- net MCT.PWM: now also Q2.3 (D); no longer R25.1
- net at J8.3 (Pin_3), R14.1: now also U18.7
- new net: Q2.2 (S), R25.1
- new net BLDC.PWM_EN: Q2.1 (G), R36.2
Other:
- moved on the sheet: R14
