File: Hardware/DriverMotor.kicad_pcb (KiCad board)
At the start: 2 copper layers, 103 parts, among them J1 Conn_02x03_Odd_Even, J10 Screw_Terminal_01x04, J11 Screw_Terminal_01x04, J12 Screw_Terminal_01x04, J13 Screw_Terminal_01x02, J2 Screw_Terminal_01x02, J3 Conn_02x04_Counter_Clockwise, J4 Screw_Terminal_01x04, J5 Screw_Terminal_01x03, J6 Screw_Terminal_01x03, J7 Conn_01x03_Pin, J8 Conn_01x03_Pin, U10 MCT8316, U11 B0505S, U12 ISO7721DR, U13 EL817, U14 EL817, U15 EL817, U16 TJA1051T, U3 XL1509-5.0, U5 MCU_STM32F103C8Tx, U7 HCPL-2631, U8 HCPL-2631, U9 LD1117

Commit message: Add PCB
Parts:
- removed C26: 100nF, IVS_FOOTPRINTS:C_0603
- removed D3: SS54, IVS_FOOTPRINTS:Package-Diode-D_SMA
- removed D4: LED, IVS_FOOTPRINTS:LED_0603
- removed J1: Conn_02x03_Odd_Even, Connector_PinHeader_2.54mm:PinHeader_2x03_P2.54mm_Vertical
- removed J12: Screw_Terminal_01x04, Connector_PinHeader_2.54mm:PinHeader_1x04_P2.54mm_Vertical
- removed J8: Conn_01x03_Pin, Connector_PinHeader_2.54mm:PinHeader_1x03_P2.54mm_Vertical
- removed the LE1 at (214.0, 118.1)
- removed R10: 1K, IVS_FOOTPRINTS:R_0603
- removed R24: 120R, IVS_FOOTPRINTS:R_0603
- added R1: 10k, IVS_FOOTPRINTS:R_0603, F.Cu at (145.7, 114.7)
- added R2: 10k, IVS_FOOTPRINTS:R_0603, F.Cu at (145.1, 125.1)
- added R3: 10K, IVS_FOOTPRINTS:R_0603, F.Cu at (158.6, 123.7)
- added R34: 2K2, IVS_FOOTPRINTS:R_0603, F.Cu at (155.5, 110.8)
- added R4: 1M, IVS_FOOTPRINTS:R_0603, F.Cu at (152.4, 116.2)
- added S1: SolderJump3P, Jumper:SolderJumper-3_P1.3mm_Open_RoundedPad1.0x1.5mm_NumberLabels, F.Cu at (170.1, 129.3)
- added S2: SolderJump3P, Jumper:SolderJumper-3_P1.3mm_Open_RoundedPad1.0x1.5mm_NumberLabels, F.Cu at (170.0, 126.6)
- added S3: SolderJump3P, Jumper:SolderJumper-3_P1.3mm_Open_RoundedPad1.0x1.5mm_NumberLabels, F.Cu at (221.2, 115.6)
- added SW1: SW_Push, IVS_FOOTPRINTS:ButtonPush-Vert-SMD-4P-SPST_PTS810, F.Cu at (146.4, 110.8)
- added Y1: 8Mhz, IVS_FOOTPRINTS:Crystal-SMD-4P-3.2x2.6mm-3225, F.Cu at (152.3, 111.4)
- C11: value 10uF -> 4.7uF/16V; footprint IVS_FOOTPRINTS:C_0603 -> Capacitor_SMD:CP_Elec_4x5.4
- C17: value 3.3nF -> 10uF
- C23: value 4.7uF/16V -> 10uF; footprint Capacitor_SMD:CP_Elec_4x5.4 -> IVS_FOOTPRINTS:C_0603
- C25: value 10uF -> 100nF
- J10, J11: footprint Connector_PinHeader_2.54mm:PinHeader_1x04_P2.54mm_Vertical -> IVS_FOOTPRINTS:Conn-Vert-THT-4P-2.54mm-S4B_XH_SM4_TB
- J3: footprint Connector_PinHeader_2.54mm:PinHeader_2x04_P2.54mm_Vertical -> Connector_IDC:IDC-Header_2x04_P2.54mm_Vertical
- J6: footprint Connector_PinHeader_2.54mm:PinHeader_1x03_P2.54mm_Vertical -> IVS_FOOTPRINTS:Conn-Horz-SMD-3P-2.54mm-S3B_XH_SM4_TB
- J7: value Conn_01x03_Pin -> Conn_01x04_Male; footprint Connector_PinHeader_2.54mm:PinHeader_1x03_P2.54mm_Vertical -> IVS_FOOTPRINTS:Conn-Vert-THT-4P-2.54mm-S4B_XH_SM4_TB
- R11, R5, R6, R7, U2, U4: moved to F.Cu
- R8: value 1K -> 120R
- R9: value 3K1 -> 1K
- U11: value B0505S -> LD1117; footprint IVS_FOOTPRINTS:PowerSupply-DCDC-Isolate-2W-BxxxxS -> IVS_FOOTPRINTS:SOT233
- U9: value LD1117 -> B0505S; footprint IVS_FOOTPRINTS:SOT233 -> IVS_FOOTPRINTS:PowerSupply-DCDC-Isolate-2W-BxxxxS
- moved R26 110.6 mm to (222.7, 29.2)
- moved R25 110.6 mm to (222.7, 26.6)
- moved R32 110.6 mm to (222.7, 42.5)
- moved U12 110.6 mm to (249.0, 22.2)
- moved U13 110.6 mm to (229.7, 27.0)
- moved U14 110.6 mm to (229.7, 33.3)
- moved U15 110.6 mm to (229.7, 40.7)
- moved R33 110.6 mm to (222.7, 45.1)
- moved R9 99.4 mm to (280.6, 164.8)
- moved F2 87.9 mm to (141.2, 102.0), turned to 180 degrees
- moved J2 83.7 mm to (104.3, 100.0), turned to -90 degrees
- moved F1 80.5 mm to (120.0, 96.9)
- moved L2 76.9 mm to (257.6, 174.7)
- moved C15 76.9 mm to (268.0, 162.9)
- moved LE3 76.9 mm to (272.3, 170.9)
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Connections:
- net /+24V_CS renamed /Power Supply/+24V_CS
- C11 pad 1: +3V3 -> +5V
- C17 pad 1: Net-(U3-FB) -> +5V
- C17 pad 2: +5V -> GND
- C23 pad 1: +5V -> +3V3
- C24 pad 1: /+5V_CS -> /Power Supply/+5V_CS
- C25 pad 1: +5V -> +3V3
- J6 pad 1: /MCT8316/MCT_SCL -> /MCT8316/MCT_SDA
- J7 pad 1: +5V -> /MCT8316/MCT.PWM
- J7 pad 2: +5VA -> GND
- J7 pad 3: /MCT8316/BUCK -> /MCT8316/MCT.DIR
- JP1 pad 2: /MCT8316/MCT_SCL -> /MCT8316/MCT_SDA
- R16 pad 1: /BTS7960/MCU_PWM_R1 -> /BTS7960/MCU_PWM_L1
- R17 pad 1: /BTS7960/MCU_PWM_L1 -> /BTS7960/MCU_PWM_R1
- R18 pad 2: /BTS7960/PWM_DC_L1 -> /BTS7960/PWM_DC_R1
- R19 pad 2: /BTS7960/PWM_DC_R1 -> /BTS7960/PWM_DC_L1
- R25 pad 1: /MCT8316/MCU_PWM_BLDC -> /MCT8316/MCT.PWM
- R28 pad 2: /MCT8316/MCT_SCL -> /MCT8316/MCT_SDA
- R33 pad 2: /MCT8316/MCU_FG -> /MCT8316/MCT.FG
- R8 pad 1: GND -> +3V3
- R8 pad 2: Net-(U3-FB) -> Net-(LE1-Pad1)
- R9 pad 1: Net-(U3-FB) -> +5V
- R9 pad 2: +5V -> Net-(LE3-Pad1)
- U10 pad 30: /MCT8316/MCT_SCL -> /MCT8316/MCT_SDA
- U10 pad 41: (no net) -> GNDD
- U11 pad 2: +5V -> +3V3
- U12 pad 2: /MCT8316/MCU_FG -> /MCT8316/MCT.FG
- U13 pad 4: /MCT8316/MCU_FAULT -> /MCT8316/MCT.FAULT
- U14 pad 1: /MCT8316/MCU_BRAKE -> /MCT8316/MCT.BRAKE
- U15 pad 1: /MCT8316/MCU_DIR -> /MCT8316/MCT.DIR
- U16 pad 1: /TJA1050/CAN_TX -> /STM32F103/CANTX
- U16 pad 4: /TJA1050/CAN_RX -> /STM32F103/CANRX
- U5 pad 1: /STM32F103/VBAT -> unconnected-(U5-VBAT-Pad1)
- U5 pad 12: /STM32F103/MCU_PWM_R1 -> /STM32F103/MCU_PA2
- U5 pad 25: /STM32F103/MCU_FG -> /MCT8316/MCT.FG
- U5 pad 26: /STM32F103/MCU_FAULT -> /MCT8316/MCT.FAULT
- U5 pad 27: /STM32F103/MCU_BRAKE -> /MCT8316/MCT.BRAKE
- U5 pad 28: /STM32F103/MCU_DIR -> /MCT8316/MCT.DIR
- U5 pad 41: /STM32F103/MCU_PWM_BLDC -> unconnected-(U5-PB5/TIM3_CH2/SPI1_MOSI/I2C1_SMBAI-Pad41)
- U7 pad 6: /BTS7960/PWM_DC_R1 -> /BTS7960/PWM_DC_L1
- U7 pad 7: /BTS7960/PWM_DC_L1 -> /BTS7960/PWM_DC_R1
- U9 pad 2: +3V3 -> +5V
- U9 pad 3: +5V -> GNDD
Other:
- board outline added: 100 x 75 mm

Commit message: Layout PCB
Parts:
- added C26: 10uF, IVS_FOOTPRINTS:C_0603, F.Cu at (157.7, 96.3)
- added H1: MountingHole, IVS_FOOTPRINTS:MountingHole_3.2mm_M3_Pad_Via, F.Cu at (104.1, 93.0)
- added H2: MountingHole, IVS_FOOTPRINTS:MountingHole_3.2mm_M3_Pad_Via, F.Cu at (103.8, 143.3)
- added H3: MountingHole, IVS_FOOTPRINTS:MountingHole_3.2mm_M3_Pad_Via, F.Cu at (194.8, 92.5)
- added H4: MountingHole, IVS_FOOTPRINTS:MountingHole_3.2mm_M3_Pad_Via, F.Cu at (194.8, 143.5)
- added J8: Conn_01x03_Pin, IVS_FOOTPRINTS:Conn-Vert-THT-3P-2.54mm-S3B_XH_SM4_TB, F.Cu at (162.8, 91.4)
- added R10: 4k7, IVS_FOOTPRINTS:R_0603, F.Cu at (161.4, 119.9)
- added R24: 4k7, IVS_FOOTPRINTS:R_0603, F.Cu at (159.7, 119.9)
- added R36: 1K, IVS_FOOTPRINTS:R_0603, F.Cu at (154.4, 89.4)
- added R37: 1K, IVS_FOOTPRINTS:R_0603, F.Cu at (157.0, 92.2)
- added S4: SolderJump3P, Jumper:SolderJumper-3_P1.3mm_Open_RoundedPad1.0x1.5mm_NumberLabels, F.Cu at (146.0, 117.6)
- added U17: EL817, IVS_FOOTPRINTS:OptoIsolation-EL357N-G, F.Cu at (153.7, 94.5)
- C14: value 470uF/35V -> 220uF/35V; footprint IVS_FOOTPRINTS:CP-Alu-SMD-10x10.5mm -> IVS_FOOTPRINTS:CP-Alu-SMD-8x10.5mm
- J13: footprint TerminalBlock:TerminalBlock_bornier-2_P5.08mm -> IVS_FOOTPRINTS:TerminalBlock_bornier-2_P5.08mm
- J4: footprint TerminalBlock:TerminalBlock_bornier-4_P5.08mm -> IVS_FOOTPRINTS:TerminalBlock_bornier-4_P5.08mm
- J5: footprint TerminalBlock:TerminalBlock_bornier-3_P5.08mm -> IVS_FOOTPRINTS:TerminalBlock_bornier-3_P5.08mm
- moved R9 125.7 mm to (167.1, 110.7), turned to -90 degrees
- moved LE3 122.6 mm to (165.4, 110.9), turned to -90 degrees
- moved D1 122.2 mm to (169.5, 101.2), turned to 90 degrees
- moved C15 120.8 mm to (160.2, 108.5), turned to 180 degrees
- moved U12 116.2 mm to (179.8, 115.6)
- moved C14 116.0 mm to (157.7, 103.1), turned to -90 degrees
- moved L2 114.8 mm to (164.9, 107.1), turned to 180 degrees
- moved U3 114.5 mm to (165.0, 101.2), turned to 90 degrees
- moved U15 109.4 mm to (136.7, 98.3)
- moved R25 106.0 mm to (173.9, 120.7)
- moved U14 105.7 mm to (143.5, 94.5), turned to -90 degrees
- moved U13 105.5 mm to (148.6, 94.4), turned to 90 degrees
- moved R26 91.4 mm to (183.1, 111.6), turned to 180 degrees
- moved R32 90.0 mm to (190.9, 126.6), turned to -90 degrees
- moved R33 86.9 mm to (171.9, 115.6)
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Connections:
- C11 pad 1: +5V -> /BTS7960/+5V_CS
- C11 pad 2: GND -> GNDD
- C14 pad 1: +24V -> /BTS7960/+24V_CS
- C14 pad 2: GND -> GNDD
- C15 pad 1: +24V -> /BTS7960/+24V_CS
- C15 pad 2: GND -> GNDD
- C16 pad 1: +5V -> /BTS7960/+5V_CS
- C16 pad 2: GND -> GNDD
- C2 pad 1: /STM32F103/+3V3_MCU -> /MCT8316/+3V3_MCU
- C24 pad 1: /Power Supply/+5V_CS -> +5V
- C24 pad 2: GNDD -> GND
- C4 pad 1: /STM32F103/+3V3_MCU -> /MCT8316/+3V3_MCU
- C5 pad 1: /STM32F103/+3V3_MCU -> /MCT8316/+3V3_MCU
- C7 pad 1: /STM32F103/+3V3_MCU -> /MCT8316/+3V3_MCU
- D1 pad 1: GND -> GNDD
- D1 pad 2: Net-(U3-FB) -> Net-(U3-OUT)
- F1 pad 2: /Power Supply/+24V_CS -> /BTS7960/+24V_CS
- J10 pad 1: /BTS7960/EnB_1 -> /BTS7960/En.EnB_1
- J10 pad 2: /BTS7960/EnA_1 -> /BTS7960/En.EnA_1
- J11 pad 1: /BTS7960/EnB_2 -> /BTS7960/En.EnB_2
- J11 pad 2: /BTS7960/EnA_2 -> /BTS7960/En.EnA_2
- J3 pad 7: /STM32F103/+3V3_MCU -> /MCT8316/+3V3_MCU
- JP1 pad 1: /MCT8316/MCU_SDA -> /MCT8316/MCT.SDA
- JP2 pad 1: /MCT8316/MCU_SCL -> /MCT8316/MCT.SCL
- L2 pad 1: +5V -> /BTS7960/+5V_CS
- L2 pad 2: Net-(U3-FB) -> Net-(U3-OUT)
- LE2 pad 1: /STM32F103/+3V3_MCU -> /MCT8316/+3V3_MCU
- LE3 pad 2: GND -> GNDD
- R1 pad 1: /STM32F103/+3V3_MCU -> /MCT8316/+3V3_MCU
- R16 pad 1: /BTS7960/MCU_PWM_L1 -> /BTS7960/BTS.PWM_L1
- R17 pad 1: /BTS7960/MCU_PWM_R1 -> /BTS7960/BTS.PWM_R1
- R20 pad 1: /BTS7960/MCU_PWM_L2 -> /BTS7960/BTS.PWM_L2
- R21 pad 1: /BTS7960/MCU_PWM_R2 -> /BTS7960/BTS.PWM_R2
- R26 pad 1: /MCT8316/+5V_CS -> /BTS7960/+5V_CS
- R35 pad 1: /MCT8316/+5V_CS -> /BTS7960/+5V_CS
- R9 pad 1: +5V -> /BTS7960/+5V_CS
- S3 pad 1: /STM32F103/MCU_PWM_R1 -> /BTS7960/BTS.PWM_L2
- S3 pad 2: /STM32F103/MCU_PA2 -> /STM32F103/MCU_PA1
- U12 pad 8: /MCT8316/+5V_CS -> /BTS7960/+5V_CS
- U16 pad 1: /STM32F103/CANTX -> /STM32F103/CANRX
- U16 pad 4: /STM32F103/CANRX -> /STM32F103/CANTX
- U3 pad 1: +24V -> /BTS7960/+24V_CS
- U3 pad 2: Net-(U3-FB) -> Net-(U3-OUT)
- U3 pad 3: Net-(U3-FB) -> /BTS7960/+5V_CS
- U3 pad 4: GND -> GNDD
- U3 pad 5: GND -> GNDD
- U3 pad 6: GND -> GNDD
- U3 pad 7: GND -> GNDD
- U3 pad 8: GND -> GNDD
- U5 pad 10: /STM32F103/MCU_PWM_R2 -> /STM32F103/MCU_PA0
- U5 pad 11: /STM32F103/MCU_PWM_L2 -> /STM32F103/MCU_PA1
- U5 pad 12: /STM32F103/MCU_PA2 -> /BTS7960/BTS.PWM_R1
- U5 pad 13: /STM32F103/MCU_PWM_L1 -> /BTS7960/BTS.PWM_L1
- U5 pad 14: unconnected-(U5-PA4/SPI1_NSS/USART2_CK/ADC12_IN4-Pad14) -> /MCT8316/MCT.BRAKE
- U5 pad 16: /STM32F103/EnA_2 -> /BTS7960/En.EnA_2
- U5 pad 17: /STM32F103/EnB_2 -> /BTS7960/En.EnB_2
- U5 pad 24: /STM32F103/+3V3_MCU -> /MCT8316/+3V3_MCU
- U5 pad 27: /MCT8316/MCT.BRAKE -> unconnected-(U5-PB14/SPI2_MISO/USART3_RTS/TIM1_CH2N-Pad27)
- U5 pad 28: /MCT8316/MCT.DIR -> unconnected-(U5-PB15/SPI2_MOSI/TIM1_CH3N-Pad28)
- U5 pad 36: /STM32F103/+3V3_MCU -> /MCT8316/+3V3_MCU
- U5 pad 42: /STM32F103/EnA_1 -> /BTS7960/En.EnA_1
- U5 pad 43: /STM32F103/EnB_1 -> /BTS7960/En.EnB_1
- U5 pad 45: /STM32F103/MCU_SCL -> /MCT8316/MCT.SCL
- U5 pad 46: /STM32F103/MCU_SDA -> /MCT8316/MCT.SDA
- U5 pad 48: /STM32F103/+3V3_MCU -> /MCT8316/+3V3_MCU
- U5 pad 9: /STM32F103/+3V3_MCU -> /MCT8316/+3V3_MCU
- U9 pad 1: GND -> GNDD
- U9 pad 2: +5V -> /BTS7960/+5V_CS
- U9 pad 3: GNDD -> GND
- U9 pad 4: /Power Supply/+5V_CS -> +5V
Routing:
- net GNDD: vias 0 -> 8
- net /BTS7960/PWM_DC_R1: vias 0 -> 1
- net /BTS7960/+24V_M2: vias 0 -> 1
- net /BTS7960/+24V_M1: vias 0 -> 2
- net (no net): vias 0 -> 19
Other:
- board size 100 x 75 mm -> 100 x 60 mm

Commit message: Update components
Parts:
- removed J8: Conn_01x03_Pin, IVS_FOOTPRINTS:Conn-Vert-THT-3P-2.54mm-S3B_XH_SM4_TB
- removed R36: 1K, IVS_FOOTPRINTS:R_0603
- removed U13, U14, U15, U17: EL817, IVS_FOOTPRINTS:OptoIsolation-EL357N-G
- added J1: Conn_01x03_Pin, IVS_FOOTPRINTS:Conn-Vert-THT-3P-2.54mm-S3B_XH_SM4_TB, F.Cu at (158.6, 92.2)
- added R38: 1K, IVS_FOOTPRINTS:R_0603, F.Cu at (153.6, 97.3)
- added U18: ~, IVS_FOOTPRINTS:SOIC-16W_5.3x10.2mm_P1.27mm, F.Cu at (146.9, 96.7)
- C11: footprint Capacitor_SMD:CP_Elec_4x5.4 -> IVS_FOOTPRINTS:C_1206
- C21: footprint IVS_FOOTPRINTS:CP-Tantalum-EIA-3528-15-AVX-H -> Capacitor_Tantalum_SMD:CP_EIA-7343-15_Kemet-W_Pad2.25x2.55mm_HandSolder
- C24: value 10uF/16V -> 10uF/10V; footprint Capacitor_SMD:CP_Elec_4x5.4 -> IVS_FOOTPRINTS:C_1206
- L2: footprint Inductor_SMD:L_1812_4532Metric -> Inductor_SMD:L_7.3x7.3_H4.5
- moved L2 29.8 mm to (194.2, 101.2), turned to -90 degrees
- moved JP3 15.1 mm to (173.1, 135.2), turned to 0 degrees
- moved C18 7.16 mm to (185.0, 122.0), turned to 90 degrees
- moved R37 6.08 mm to (151.0, 91.1), turned to 180 degrees
- moved C27 5.14 mm to (166.4, 127.3), turned to 180 degrees
- moved F4 3.92 mm to (133.0, 121.4), turned to -90 degrees
- moved C28 3.73 mm to (169.6, 137.1)
- moved C1 3.11 mm to (146.7, 105.4)
- moved U16 3.10 mm to (168.1, 132.5), turned to -90 degrees
- moved SW1 3.06 mm to (146.6, 109.2)
- moved R1 3.06 mm to (146.0, 113.1)
- moved R25 2.88 mm to (174.1, 117.8), turned to 90 degrees
- moved J13 2.85 mm to (164.0, 143.9)
- moved C22 2.72 mm to (179.0, 124.6)
- moved C29 2.63 mm to (166.4, 137.1), turned to 180 degrees
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Connections:
- C26 pad 2: /BTS7960/+24V_CS -> /MCT8316/+24V_CS
- J13 pad 1: /TJA1050/CANH -> /TJA1050/CANL
- J13 pad 2: /TJA1050/CANL -> /TJA1050/CANH
Routing:
- net /BTS7960/+24V_CS: track 0.00 -> 58.0 mm
- net /BTS7960/+24V_M1: track 0.00 -> 39.4 mm
- net +24V: track 0.00 -> 37.2 mm
- net /BTS7960/+5V_CS: track 0.00 -> 35.1 mm
- net /BTS7960/Motor_L1: track 0.00 -> 27.1 mm
- net /BTS7960/+24V_M2: track 0.00 -> 23.6 mm, vias 1 -> 2
- net /BTS7960/Motor_R2: track 0.00 -> 22.5 mm
- net /BTS7960/Motor_R1: track 0.00 -> 22.3 mm
- net /BTS7960/Motor_L2: track 0.00 -> 19.8 mm
- net GNDD: track 0.00 -> 15.8 mm
- net /BTS7960/PWM_DC_R1: track 0.00 -> 11.8 mm
- net /BTS7960/PWM_DC_L1: track 0.00 -> 9.70 mm
- net GND: track 0.00 -> 5.10 mm, vias 0 -> 1
- net Net-(U1-SR): track 0.00 -> 4.29 mm
- net Net-(U1-IS): track 0.00 -> 4.09 mm
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
Commit message: Update Encoder
Parts:
- moved C26 3.13 mm to (160.2, 96.3), turned to 0 degrees
- moved J6 1.67 mm to (194.0, 115.1)
- moved C15 1.07 mm to (161.0, 109.2)
- moved U9 1.07 mm to (185.9, 96.3)
- moved J7 0.87 mm to (133.9, 91.9)
- moved L2 0.78 mm to (194.3, 102.0)
- moved C14 0.76 mm to (158.3, 103.8)
- moved J1 0.51 mm to (158.8, 91.7), turned to -90 degrees
- moved R37 0.45 mm to (151.0, 91.6)
- moved U18 0.45 mm to (146.9, 97.2)
- moved R38 0.45 mm to (153.6, 97.7)
Routing:
- net Net-(R37-Pad2): track 0.00 -> 2.15 mm
- net GND: track 5.10 -> 6.79 mm, vias 1 -> 2
Changed lines of the file:
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@@
   )
   (footprint "IVS_FOOTPRINTS:Conn-Vert-THT-4P-2.54mm-S4B_XH_SM4_TB" (layer "F.Cu")
-    (at 134.314748 91.17 -90)
+    (at 133.92 91.94 -90)
     (tags "XH 2.54 ")
     (property "Sheetfile" "MCT8316.kicad_sch")
@@
   )
   (footprint "IVS_FOOTPRINTS:R_0603" (layer "F.Cu")
-    (at 150.99 91.11 180)
+    (at 150.955252 91.56 180)
     (property "Sheetfile" "MCT8316.kicad_sch")
     (property "Sheetname" "MCT8316")
@@
   )
   (footprint "IVS_FOOTPRINTS:SOIC-16W_5.3x10.2mm_P1.27mm" (layer "F.Cu")
-    (at 146.944748 96.72 90)
+    (at 146.91 97.17 90)
     (descr "16-Lead Plastic Small Outline (SO) - Wide, 5.3 mm Body (http://www.ti.com/lit/ml/msop002a/msop002a.pdf)")
     (tags "SOIC 1.27")
@@
     (property "Sheetname" "MCT8316")
     (attr smd)
-    (fp_text reference "U18" (at -5.35 -3.9) (layer "F.SilkS")
+    (fp_text reference "U18" (at 0.03 -0.04) (layer "F.SilkS")
         (effects (font (size 0.6 0.6) (thickness 0.15)))
     )
@@
     (property "ki_keywords" "solder jumper SPST")
     (attr exclude_from_pos_files)
-    (fp_text reference "JP1" (at -4.622 -2.069 -90) (layer "F.SilkS")
+    (fp_text reference "JP1" (at -2.7 -0.112 -90) (layer "F.SilkS")
         (effects (font (size 0.6 0.6) (thickness 0.15)))
     )
@@
   )
   (footprint "IVS_FOOTPRINTS:Conn-Vert-THT-3P-2.54mm-S3B_XH_SM4_TB" (layer "F.Cu")
-    (at 158.61 92.23 90)
+    (at 158.75 91.74 -90)
     (tags "XH 2.54 ")
     (property "Sheetfile" "MCT8316.kicad_sch")
@@
     (property "ki_keywords" "connector")
     (attr through_hole)
-    (fp_text reference "J1" (at 1.5 4.04 90 unlocked) (layer "F.SilkS") hide
+    (fp_text reference "J1" (at 1.5 4.04 -90 unlocked) (layer "F.SilkS") hide
         (effects (font (size 0.8 0.8) (thickness 0.3)))
     )
-    (fp_text value "Conn_01x03_Pin" (at 0 7.4 90 unlocked) (layer "F.Fab")
+    (fp_text value "Conn_01x03_Pin" (at 0 7.4 -90 unlocked) (layer "F.Fab")
         (effects (font (size 1 1) (thickness 0.15)))
     )
@@
     (fp_rect (start -3.02 -5.12) (end 3.59 5.06)
       (stroke (width 0.05) (type solid)) (fill none) (layer "F.CrtYd"))
-    (pad "1" thru_hole rect (at 0 -2.54 90) (size 3 1.5) (drill 1) (layers "*.Cu" "*.Mask")
+    (pad "1" thru_hole rect (at 0 -2.54 270) (size 3 1.5) (drill 1) (layers "*.Cu" "*.Mask")
       (net 108 "/MCT8316/+24V_CS") (pinfunction "Pin_1") (pintype "passive"))
-    (pad "2" thru_hole oval (at 0 0 90) (size 3 1.5) (drill 1) (layers "*.Cu" "*.Mask")
+    (pad "2" thru_hole oval (at 0 0 270) (size 3 1.5) (drill 1) (layers "*.Cu" "*.Mask")
       (net 107 "Net-(J1-Pin_2)") (pinfunction "Pin_2") (pintype "passive"))
-    (pad "3" thru_hole oval (at 0 2.54 90) (size 3 1.5) (drill 1) (layers "*.Cu" "*.Mask")
+    (pad "3" thru_hole oval (at 0 2.54 270) (size 3 1.5) (drill 1) (layers "*.Cu" "*.Mask")
       (net 109 "Net-(J1-Pin_3)") (pinfunction "Pin_3") (pintype "passive"))
     (model "E:/IoT_Lab/3D/Connector/XH_2.54/Thru Vertical/JST - XH - Thru (V) - 3Pin - 2.54mm.stp"
@@
   )
   (footprint "IVS_FOOTPRINTS:C_0603" (layer "F.Cu")
-    (at 157.02 96.165 180)
+    (at 160.15 96.33)
     (property "Sheetfile" "MCT8316.kicad_sch")
     (property "Sheetname" "MCT8316")
@@
         (effects (font (size 0.6 0.6) (thickness 0.15) bold))
     )
-    (fp_text value "10uF" (at 0 0.95 180 unlocked) (layer "F.Fab")
+    (fp_text value "10uF" (at 0 0.95 unlocked) (layer "F.Fab")
         (effects (font (size 1 1) (thickness 0.15)))
     )
-    (fp_text user "${REFERENCE}" (at 0 0 180 unlocked) (layer "F.Fab")
+    (fp_text user "${REFERENCE}" (at 0 0 unlocked) (layer "F.Fab")
         (effects (font (size 1 1) (thickness 0.15)))
     )
@@
     (fp_line (start 0.8 0.41) (end -0.8 0.41)
       (stroke (width 0.1) (type solid)) (layer "F.Fab"))
-    (pad "1" smd roundrect (at -0.775 0 180) (size 0.85 0.9) (layers "F.Cu" "F.Paste" "F.Mask") (roundrect_rratio 0.15)
+    (pad "1" smd roundrect (at -0.775 0) (size 0.85 0.9) (layers "F.Cu" "F.Paste" "F.Mask") (roundrect_rratio 0.15)
       (net 107 "Net-(J1-Pin_2)") (pintype "passive"))
-    (pad "2" smd roundrect (at 0.775 0 180) (size 0.85 0.9) (layers "F.Cu" "F.Paste" "F.Mask") (roundrect_rratio 0.15)
+    (pad "2" smd roundrect (at 0.775 0) (size 0.85 0.9) (layers "F.Cu" "F.Paste" "F.Mask") (roundrect_rratio 0.15)
       (net 108 "/MCT8316/+24V_CS") (pintype "passive"))
     (model "${IOTVISION_3D}/Capacitor/Cap_SMD/CAP/csmd-0603_l1-6_w0-81_h0-86.stp"
@@
   )
   (footprint "IVS_FOOTPRINTS:PowerSupply-DCDC-Isolate-2W-BxxxxS" (layer "F.Cu")
-    (at 186.949 96.243 180)
+    (at 185.88 96.27 180)
     (property "Field2" "")
     (property "Sheetfile" "Power_Supply.kicad_sch")
@@
   )
   (footprint "IVS_FOOTPRINTS:C_0603" (layer "F.Cu")
-    (at 160.2115 108.489125 180)
+    (at 160.98 109.24 180)
     (property "Field2" "")
     (property "Sheetfile" "Power_Supply.kicad_sch")
@@
   )
   (footprint "IVS_FOOTPRINTS:CP-Alu-SMD-8x10.5mm" (layer "F.Cu")
-    (at 157.97 103.17 -90)
+    (at 158.34 103.83 -90)
     (property "Field2" "")
     (property "Sheetfile" "Power_Supply.kicad_sch")
@@
   )
   (footprint "IVS_FOOTPRINTS:R_0603" (layer "F.Cu")
-    (at 153.61 97.29 90)
+    (at 153.575252 97.74 90)
     (property "Sheetfile" "MCT8316.kicad_sch")
     (property "Sheetname" "MCT8316")
@@
     (property "ki_keywords" "R res resistor")
     (attr smd)
-    (fp_text reference "R38" (at 0.05 1.34 270 unlocked) (layer "F.SilkS")
+    (fp_text reference "R38" (at -2.51 -0.335252 270 unlocked) (layer "F.SilkS")
         (effects (font (size 0.6 0.6) (thickness 0.15) bold))
     )
@@
   )
   (footprint "IVS_FOOTPRINTS:Conn-Horz-SMD-3P-2.54mm-S3B_XH_SM4_TB" (layer "F.Cu")
-    (at 193.88 113.42 90)
+    (at 193.98 115.09 90)
     (descr "JST-XH-2.54-SMD")
     (property "Sheetfile" "MCT8316.kicad_sch")
@@
   )
   (footprint "Inductor_SMD:L_7.3x7.3_H4.5" (layer "F.Cu")
-    (at 194.18 101.22 -90)
+    (at 194.34 101.98 -90)
     (descr "Choke, SMD, 7.3x7.3mm 4.5mm height")
     (tags "Choke SMD")
@@
     (property "ki_keywords" "inductor choke coil reactor magnetic")
     (attr smd)
-    (fp_text reference "L2" (at 5.16 -3.16 90) (layer "F.SilkS")
+    (fp_text reference "L2" (at -4.91 3.36) (layer "F.SilkS")
         (effects (font (size 1 1) (thickness 0.15)))
     )
@@
   (via blind (at 150.1 112.522) (size 0.6) (drill 0.3) (layers "F.Cu" "B.Cu") (net 0))
   (via blind (at 150.1 109.474) (size 0.6) (drill 0.3) (layers "F.Cu" "B.Cu") (net 0))
+  (segment (start 135.19 91.94) (end 135.19 90.02) (width 0.25) (layer "F.Cu") (net 1))
   (segment (start 125.82 93.726) (end 120.948 93.726) (width 1) (layer "F.Cu") (net 1))
-  (segment (start 133.477 99.568) (end 133.2475 99.568) (width 0.25) (layer "F.Cu") (net 1))
   (via (at 125.82 93.726) (size 0.8) (drill 0.4) (layers "F.Cu" "B.Cu") (net 1))
+  (via (at 135.19 90.02) (size 0.5) (drill 0.3) (layers "F.Cu" "B.Cu") (net 1))
   (segment (start 126.895 143.6325) (end 127.05 143.4775) (width 0.5) (layer "F.Cu") (net 5))
   (segment (start 127.035 118.6525) (end 127.1 118.5875) (width 0.5) (layer "F.Cu") (net 5))
@@
   (segment (start 123.48 144.9025) (end 126.925 144.9025) (width 0.25) (layer "F.Cu") (net 66))
   (segment (start 126.925 144.9025) (end 127.05 145.0275) (width 0.25) (layer "F.Cu") (net 66))
+  (segment (start 150.180252 93.574748) (end 150.085 93.67) (width 0.25) (layer "F.Cu") (net 110))
+  (segment (start 150.180252 91.56) (end 150.180252 93.574748) (width 0.25) (layer "F.Cu") (net 110))
   (zone (net 0) (net_name "") (layers "F&B.Cu") (hatch edge 0.5)
     (connect_pads (clearance 0))
