File: Hardware/DriverMotor.kicad_pcb (KiCad board)
At the start: 2 copper layers, 100 x 60 mm, 113 parts, among them J1 Conn_01x03_Pin, J10 Screw_Terminal_01x04, J11 Screw_Terminal_01x04, J13 Screw_Terminal_01x02, J2 Screw_Terminal_01x02, J3 Conn_02x04_Counter_Clockwise, J4 Screw_Terminal_01x04, J5 Screw_Terminal_01x03, J6 Screw_Terminal_01x03, J7 Conn_01x04_Male, SW1 SW_Push, U10 MCT8316, U11 LD1117, U12 ISO7721DR, U16 TJA1051T, U3 XL1509-5.0, U5 MCU_STM32F103C8Tx, U7 HCPL-2631, U8 HCPL-2631, U9 B0505S, Y1 8Mhz

Commit message: Fix bug schematic
Parts:
- removed J3: Conn_02x04_Counter_Clockwise, Connector_IDC:IDC-Header_2x04_P2.54mm_Vertical
- added J12: Conn_01x04_Male, Connector_PinHeader_2.54mm:PinHeader_1x04_P2.54mm_Vertical, F.Cu at (165.8, 90.6)
- added J8: Conn_02x04_Odd_Even, Connector_IDC:IDC-Header_2x04_P2.54mm_Vertical, F.Cu at (157.2, 133.4)
- added J9: Conn_01x07_Pin, Connector_PinHeader_2.54mm:PinHeader_1x07_P2.54mm_Vertical, F.Cu at (188.3, 101.2)
- added TP1: TestPoint, IVS_FOOTPRINTS:TestPoint_Pad_D1.0mm, F.Cu at (190.6, 121.9)
- added TP2: TestPoint, IVS_FOOTPRINTS:TestPoint_Pad_D1.0mm, F.Cu at (188.7, 121.9)
- added TP3: TestPoint, IVS_FOOTPRINTS:TestPoint_Pad_D1.0mm, F.Cu at (186.9, 121.9)
- C12, C18, C19, C22: footprint IVS_FOOTPRINTS:C_0603 -> IVS_FOOTPRINTS:C_0805
- J6: footprint IVS_FOOTPRINTS:Conn-Horz-SMD-3P-2.54mm-S3B_XH_SM4_TB -> IVS_FOOTPRINTS:XH_3P_2.54mm_Vertical
- moved D1 2.82 mm to (170.8, 105.0)
- moved U3 2.82 mm to (165.7, 104.9)
- moved R35 0.91 mm to (190.6, 134.3), turned to -90 degrees
- moved U18 0.60 mm to (146.4, 97.4), turned to -90 degrees
- moved J6 0.55 mm to (194.1, 115.6)
- moved L2 0.55 mm to (194.4, 102.5)
- moved J1 0.50 mm to (158.2, 91.7)
Connections:
- C26 pad 2: /MCT8316/+24V_CS -> /BTS7960/+24V_CS
- J1 pad 1: /MCT8316/+24V_CS -> /BTS7960/+24V_CS
- J10 pad 3: /BTS7960/+5V_CS -> +5V
- J10 pad 4: GNDD -> GND
- J11 pad 3: /BTS7960/+5V_CS -> +5V
- J11 pad 4: GNDD -> GND
- R38 pad 1: Net-(R38-Pad1) -> /MCT8316/PA5
- U10 pad 37: unconnected-(U10-DACOUT1-Pad37) -> /MCT8316/MCT_DACOUT1
- U10 pad 38: unconnected-(U10-DACOUT2-Pad38) -> /MCT8316/MCT_DACOUT2
- U18 pad 10: Net-(R37-Pad2) -> /MCT8316/+3V3_MCU
- U18 pad 7: /MCT8316/+3V3_MCU -> Net-(R37-Pad2)
- U18 pad 8: Net-(R38-Pad1) -> GNDD
- U18 pad 9: GNDD -> /MCT8316/PA5
- U5 pad 15: unconnected-(U5-PA5/SPI1_SCK/ADC12_IN5-Pad15) -> /MCT8316/PA5
- U5 pad 18: unconnected-(U5-PB0/ADC12_IN8/TIM3_CH3/TIM1_CH2N-Pad18) -> /STM32F103/PB0
- U5 pad 19: unconnected-(U5-PB1/ADC12_IN9/TIM3_CH4/TIM1_CH3N-Pad19) -> /STM32F103/PB1
- U5 pad 27: unconnected-(U5-PB14/SPI2_MISO/USART3_RTS/TIM1_CH2N-Pad27) -> /STM32F103/PB14
- U5 pad 28: unconnected-(U5-PB15/SPI2_MOSI/TIM1_CH3N-Pad28) -> /STM32F103/PB15
- U5 pad 29: unconnected-(U5-PA8/USART1_CK/TIM1_CH1/MCO-Pad29) -> /STM32F103/PA8
- U5 pad 30: unconnected-(U5-PA9/USART1_TX/TIM1_CH2-Pad30) -> /STM32F103/PA9
- U5 pad 31: unconnected-(U5-PA10/USART1_RX/TIM1_CH3-Pad31) -> /STM32F103/PA10
- U5 pad 38: unconnected-(U5-PA15/JTDI-Pad38) -> /STM32F103/PA15
- U5 pad 39: unconnected-(U5-PB3/JTDO/TIM2_CH2/TRACESWO/SPI1_SCK-Pad39) -> /STM32F103/PB3
- U5 pad 40: unconnected-(U5-PB4/JNTRST/TIM3_CH1/SPI1_MISO-Pad40) -> /STM32F103/PB4
- U5 pad 41: unconnected-(U5-PB5/TIM3_CH2/SPI1_MOSI/I2C1_SMBAI-Pad41) -> /STM32F103/PB5
Routing:
- net Net-(R37-Pad2): track 2.15 -> 0.00 mm

Commit message: Layout track part 2
Parts:
- removed TP1, TP2, TP3: TestPoint, IVS_FOOTPRINTS:TestPoint_Pad_D1.0mm
- added C30: 100nF, IVS_FOOTPRINTS:C_0603, F.Cu at (100.5, 96.1)
- added DACOUT1: TestPoint, IVS_FOOTPRINTS:TestPoint_Pad_D1.0mm, F.Cu at (174.6, 119.2)
- added DACOUT2: TestPoint, IVS_FOOTPRINTS:TestPoint_Pad_D1.0mm, F.Cu at (174.6, 121.0)
- added G***: LOGO, IVS_FOOTPRINTS:Logo_Phap_F, F.Cu at (75.9, 140.7)
- added Q1: P_Mosfet, Package_TO_SOT_SMD:TO-252-2, F.Cu at (105.5, 93.3)
- added R36: 1K, IVS_FOOTPRINTS:R_0603, B.Cu at (172.5, 141.7)
- added R39: 2K, IVS_FOOTPRINTS:R_0603, B.Cu at (170.6, 141.7)
- added R40: 2K, IVS_FOOTPRINTS:R_0603, B.Cu at (167.0, 141.7)
- added R41: 1K, IVS_FOOTPRINTS:R_0603, B.Cu at (168.8, 141.7)
- added R42: 2K, IVS_FOOTPRINTS:R_0603, B.Cu at (159.7, 141.7)
- added R43: 2K, IVS_FOOTPRINTS:R_0603, B.Cu at (154.2, 141.7)
- added R44: 1K, IVS_FOOTPRINTS:R_0603, B.Cu at (157.8, 141.7)
- added R45: 1K, IVS_FOOTPRINTS:R_0603, B.Cu at (156.0, 141.7)
- added R46: 100k, IVS_FOOTPRINTS:R_0603, F.Cu at (100.5, 99.3)
- added SOX1: TestPoint, IVS_FOOTPRINTS:TestPoint_Pad_D1.0mm, F.Cu at (174.7, 117.5)
- added Z1: 15V, IVS_FOOTPRINTS:Package-Diode-D_MiniMELF, F.Cu at (103.0, 102.8)
- C11, C24, C26, R37: moved to B.Cu
- C15: footprint IVS_FOOTPRINTS:C_0603 -> IVS_FOOTPRINTS:C_1206
- J12: footprint Connector_PinHeader_2.54mm:PinHeader_1x04_P2.54mm_Vertical -> IVS_FOOTPRINTS:Conn-Horz-SMD-4P-2.54mm-PinHeader; moved to B.Cu
- J6: footprint IVS_FOOTPRINTS:XH_3P_2.54mm_Vertical -> Connector_PinHeader_2.54mm:PinHeader_1x03_P2.54mm_Vertical
- J9: footprint Connector_PinHeader_2.54mm:PinHeader_1x07_P2.54mm_Vertical -> IVS_FOOTPRINTS:Conn-Horz-SMD-7P-2.54mm-PinHeader; moved to B.Cu
- R8: value 120R -> 1k
- moved J7 62.7 mm to (195.0, 105.8), turned to 0 degrees
- moved J12 56.6 mm to (196.4, 138.2)
- moved L2 46.0 mm to (152.5, 83.6), turned to 180 degrees
- moved F2 42.2 mm to (179.3, 93.2), turned to 0 degrees
- moved J9 40.9 mm to (169.6, 137.6), turned to 90 degrees
- moved R37 40.0 mm to (190.8, 95.9), turned to -90 degrees
- moved J1 36.8 mm to (195.0, 93.7), turned to 0 degrees
- moved R8 36.6 mm to (150.6, 94.5), turned to 180 degrees
- moved LE1 34.1 mm to (150.6, 96.2), turned to 0 degrees
- moved U3 32.4 mm to (142.1, 82.8), turned to 180 degrees
- moved C14 31.2 mm to (133.5, 84.9), turned to 90 degrees
- moved C26 30.9 mm to (190.8, 92.1), turned to 90 degrees
- moved U2 30.0 mm to (122.7, 101.4)
- moved R22 30.0 mm to (134.3, 103.3)
- moved C8 30.0 mm to (136.0, 103.3)
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Connections:
- net Net-(U10-DVDD) renamed /MCT8316/DVDD
- net Net-(U10-SW_BK) renamed /MCT8316/SW_BUCK
- net Net-(U3-OUT) renamed /Power Supply/XL1509_OUT
- net Net-(U5-PC13/TAMPER-RTC) renamed /STM32F103/PC13
- C19 pad 2: Net-(C19-Pad2) -> /MCT8316/VM
- C20 pad 2: Net-(C19-Pad2) -> /MCT8316/VM
- C21 pad 1: Net-(C19-Pad2) -> /MCT8316/VM
- C22 pad 1: Net-(U10-GND_BK) -> GNDD
- F1 pad 1: +24V -> /Power Supply/S
- F2 pad 1: Net-(C19-Pad2) -> /BTS7960/+24V_CS
- F2 pad 2: +24V -> /MCT8316/VM
- J10 pad 1: /BTS7960/En.EnB_1 -> Net-(J10-Pin_1)
- J10 pad 2: /BTS7960/En.EnA_1 -> Net-(J10-Pin_2)
- J11 pad 1: /BTS7960/En.EnB_2 -> Net-(J11-Pin_1)
- J11 pad 2: /BTS7960/En.EnA_2 -> Net-(J11-Pin_2)
- J2 pad 2: GND -> GNDD
- J4 pad 1: /BTS7960/Motor_L1 -> /BTS7960/Motor_L2
- J4 pad 2: /BTS7960/Motor_R1 -> /BTS7960/Motor_R2
- J4 pad 3: /BTS7960/Motor_L2 -> /BTS7960/Motor_L1
- J4 pad 4: /BTS7960/Motor_R2 -> /BTS7960/Motor_R1
- J9 pad 1: /STM32F103/PB0 -> /STM32F103/PB5
- J9 pad 2: /STM32F103/PB1 -> /STM32F103/PB4
- J9 pad 4: /STM32F103/PB4 -> /STM32F103/PB15
- J9 pad 5: /STM32F103/PB5 -> /STM32F103/PB14
- J9 pad 6: /STM32F103/PB14 -> /STM32F103/PB0
- J9 pad 7: /STM32F103/PB15 -> /STM32F103/PB1
- R16 pad 1: /BTS7960/BTS.PWM_L1 -> /BTS7960/BTS.PWM_R1
- R17 pad 1: /BTS7960/BTS.PWM_R1 -> /BTS7960/BTS.PWM_L1
- R18 pad 2: /BTS7960/PWM_DC_R1 -> /BTS7960/PWM_DC_L1
- R19 pad 2: /BTS7960/PWM_DC_L1 -> /BTS7960/PWM_DC_R1
- U10 pad 10: Net-(C19-Pad2) -> /MCT8316/VM
- U10 pad 11: Net-(C19-Pad2) -> /MCT8316/VM
- U10 pad 26: /MCT8316/AVDD -> GNDD
- U10 pad 27: GNDD -> /MCT8316/AVDD
- U10 pad 4: Net-(U10-GND_BK) -> GNDD
- U10 pad 9: Net-(C19-Pad2) -> /MCT8316/VM
- U7 pad 6: /BTS7960/PWM_DC_L1 -> /BTS7960/PWM_DC_R1
- U7 pad 7: /BTS7960/PWM_DC_R1 -> /BTS7960/PWM_DC_L1
Routing:
- net +5V: track 0.00 -> 139.2 mm, vias 0 -> 8
- net /MCT8316/+3V3_MCU: track 0.00 -> 105.7 mm, vias 0 -> 5
- net GNDD: track 15.8 -> 104.6 mm, vias 8 -> 13
- net /MCT8316/MCT.FAULT: track 0.00 -> 61.5 mm, vias 0 -> 2
- net /MCT8316/MCT.PWM: track 0.00 -> 58.4 mm, vias 0 -> 2
- net /MCT8316/MCT.DIR: track 0.00 -> 58.3 mm, vias 0 -> 2
- net /MCT8316/MCT.FG: track 0.00 -> 48.7 mm, vias 0 -> 2
- net /MCT8316/VM: track 0.00 -> 48.5 mm, vias 0 -> 6
- net +5VA: track 0.00 -> 42.6 mm, vias 0 -> 2
- net /BTS7960/+24V_M1: track 39.4 -> 0.00 mm, vias 2 -> 0
- net /BTS7960/En.EnB_2: track 0.00 -> 34.8 mm, vias 0 -> 1
- net /STM32F103/CANRX: track 0.00 -> 33.8 mm, vias 0 -> 2
- net /BTS7960/En.EnA_2: track 0.00 -> 33.2 mm, vias 0 -> 1
- net /BTS7960/+24V_CS: track 58.0 -> 90.4 mm, vias 0 -> 1
- net /BTS7960/En.EnA_1: track 0.00 -> 31.6 mm, vias 0 -> 1
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- added copper zone on F.Cu, net +24V
- added copper zone on F.Cu, net +3V3
- added copper zone on F.Cu, net +5V
- added copper zone on F.Cu, net /BTS7960/+24V_CS
- added copper zone on B.Cu, net /BTS7960/+5V_CS
- added copper zone on F.Cu, net /BTS7960/+5V_CS
- added copper zone on B.Cu, net /BTS7960/Motor_L1
- added copper zone on F.Cu, net /BTS7960/Motor_L1
- added copper zone on B.Cu, net /BTS7960/Motor_L2
- added copper zone on F.Cu, net /BTS7960/Motor_L2
- added copper zone on B.Cu, net /BTS7960/Motor_R1
- added copper zone on F.Cu, net /BTS7960/Motor_R1
- added copper zone on B.Cu, net /BTS7960/Motor_R2
- added copper zone on F.Cu, net /BTS7960/Motor_R2
- added copper zone on F.Cu, net /MCT8316/+3V3_MCU
- added copper zone on F.Cu, net /MCT8316/AVDD
- added copper zone on F.Cu, net /MCT8316/BUCK
- added copper zone on F.Cu, net /MCT8316/DVDD
- added copper zone on B.Cu, net /MCT8316/MA
- added copper zone on F.Cu, net /MCT8316/MA
- added copper zone on B.Cu, net /MCT8316/MB
- added copper zone on F.Cu, net /MCT8316/MB
- added copper zone on B.Cu, net /MCT8316/MC
- added copper zone on F.Cu, net /MCT8316/MC
- added copper zone on F.Cu, net /MCT8316/SW_BUCK
- added copper zone on B.Cu, net /MCT8316/VM
- added copper zone on F.Cu, net /MCT8316/VM
- added copper zone on F.Cu, net /Power Supply/S
- added copper zone on F.Cu, net /Power Supply/XL1509_OUT
- added copper zone on F.Cu, net GNDD
Other:
- board size 100 x 60 mm -> 100 x 70 mm

Commit message: Complete layout board
Parts:
- added G***: LOGO, LOGO, B.Cu at (149.5, 84.0)
- G***: moved to B.Cu
- moved G*** 98.6 mm to (157.1, 84.7), turned to 180 degrees
- moved R18 14.2 mm to (134.8, 131.0)
- moved R19 13.4 mm to (135.6, 144.8)
- moved Z1 1.88 mm to (104.9, 102.7)
- moved H4 1.41 mm to (194.6, 144.8)
- moved C25 1.08 mm to (157.7, 101.9)
- moved U11 1.08 mm to (158.3, 96.6)
- moved C23 1.08 mm to (157.7, 103.7)
- moved R11 1.01 mm to (135.7, 112.7)
- moved H2 1.00 mm to (103.5, 144.8)
- moved H3 1.00 mm to (194.6, 83.8)
- moved F4 0.99 mm to (139.5, 91.6)
- moved R7 0.93 mm to (135.7, 114.4)
- moved R14 0.87 mm to (135.6, 126.4)
- moved R23 0.87 mm to (135.0, 117.2)
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- renumbered JP2 to SCL/PB8, JP1 to SDA/PB9
Connections:
- J7 pad 1: /MCT8316/MCT.PWM -> /MCT8316/PWM_BLDC
Routing:
- net /BTS7960/+5V_CS: track 53.5 -> 252.0 mm, vias 5 -> 11
- net GND: track 35.7 -> 230.5 mm, vias 33 -> 59
- net GNDD: track 104.6 -> 255.1 mm, vias 13 -> 48
- net /MCT8316/MCT.BRAKE: track 0.00 -> 88.2 mm, vias 0 -> 5
- net /MCT8316/PA5: track 0.00 -> 63.6 mm, vias 0 -> 4
- net /MCT8316/+3V3_MCU: track 105.7 -> 163.8 mm, vias 5 -> 11
- net /STM32F103/PA8: track 1.89 -> 58.0 mm, vias 1 -> 3
- net /STM32F103/PA9: track 0.00 -> 54.3 mm, vias 0 -> 3
- net /STM32F103/PA10: track 0.00 -> 51.6 mm, vias 0 -> 3
- net /STM32F103/PA15: track 1.44 -> 46.2 mm, vias 1 -> 3
- net /MCT8316/PWM_BLDC: track 0.00 -> 35.7 mm
- net /BTS7960/PWM_DC_R2: track 0.00 -> 32.7 mm, vias 0 -> 1
- net /MCT8316/MCT_DIR: track 0.00 -> 31.6 mm, vias 0 -> 2
- net /MCT8316/MCT_FAULT: track 14.4 -> 43.5 mm, vias 2 -> 3
- net /MCT8316/MCT_BRAKE: track 0.00 -> 28.4 mm, vias 0 -> 2
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- added copper zone on B.Cu, net /BTS7960/+24V_M1
- added copper zone on F.Cu, net /BTS7960/+24V_M1
- added copper zone on B.Cu, net /BTS7960/+24V_M2
- added copper zone on F.Cu, net /BTS7960/+24V_M2
- added copper zone on B.Cu, net GND
- added copper zone on F.Cu, net GND
- added copper zone on B.Cu, net GNDD
Other:
- outline, holes or cut-outs redrawn
- board text added: "+24V"
- board text added: "120R"
- board text added: "24V"
- board text added: "3.3V"
- board text added: "5V"
- board text added: "A1"
- board text added: "A2"
- board text added: "B0505"
- board text added: "B1"
- board text added: "B2"
- board text added: "BLDC"
- board text added: "BRAKE PA4"
- board text added: "CANH"
- board text added: "CANL"
- board text added: "DC"
- board text added: "DIR PA0"
- board text added: "G"
- board text added: "GND"
- board text added: "IN"
- board text added: "LD1117"
- board text added: "MA"
- board text added: "MB"
- board text added: "MC"
- board text added: "MCT_BK"
- board text added: "MCT_LDO"
- board text added: "MOTOR1"
- board text added: "MOTOR2"
- board text added: "Motor Driver V1.0.0"
- board text added: "PA0"
- board text added: "PA1"
- board text added: "PA10"
- board text added: "PA15"
- board text added: "PA2"
- board text added: "PA3"
- board text added: "PA8"
- board text added: "PA9"
- board text added: "PB0"
- board text added: "PB1"
- board text added: "PB14"
- board text added: "PB15"
- board text added: "PB3"
- board text added: "PB4"
- board text added: "PB5"
- board text added: "PWM PA1"
- board text added: "RESET"
- board text added: "SCL"
- board text added: "SDA"
- board text added: "ST-Link Header"

Commit message: Update README
Changed lines of the file:
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@@
     (property "ki_keywords" "screw terminal")
     (attr through_hole)
-    (fp_text reference "J2" (at -5.67 -0.015) (layer "F.SilkS")
+    (fp_text reference "J2" (at 13.335 -0.015) (layer "F.SilkS")
         (effects (font (size 1 1) (thickness 0.15)))
     )
-    (fp_text value "Screw_Terminal_01x02" (at 3.6 5.4) (layer "F.Fab")
+    (fp_text value "Screw_Terminal_01x02" (at 4.065 5.4) (layer "F.Fab")
         (effects (font (size 1 1) (thickness 0.15)))
     )
-    (fp_text user "${REFERENCE}" (at 3.6 0.05) (layer "F.Fab")
+    (fp_text user "${REFERENCE}" (at 4.065 0.05) (layer "F.Fab")
         (effects (font (size 1 1) (thickness 0.15)))
     )
-    (fp_line (start -4.25 -1.6) (end -4.25 1.55)
+    (fp_line (start -3.785 -4.15) (end 9.065 -4.15)
       (stroke (width 0.12) (type solid)) (layer "F.SilkS"))
-    (fp_line (start -4.25 1.55) (end -1.4 4.15)
+    (fp_line (start -3.785 4.15) (end -3.785 -4.15)
       (stroke (width 0.12) (type solid)) (layer "F.SilkS"))
-    (fp_line (start -1.4 -4.15) (end -4.25 -1.6)
+    (fp_line (start 9.065 -4.15) (end 11.915 -1.6)
       (stroke (width 0.12) (type solid)) (layer "F.SilkS"))
-    (fp_line (start -1.4 4.15) (end 11.45 4.15)
+    (fp_line (start 9.065 4.15) (end -3.785 4.15)
       (stroke (width 0.12) (type solid)) (layer "F.SilkS"))
-    (fp_line (start 11.45 -4.15) (end -1.4 -4.15)
+    (fp_line (start 11.915 -1.6) (end 11.915 1.55)
       (stroke (width 0.12) (type solid)) (layer "F.SilkS"))
-    (fp_line (start 11.45 4.15) (end 11.45 -4.15)
+    (fp_line (start 11.915 1.55) (end 9.065 4.15)
       (stroke (width 0.12) (type solid)) (layer "F.SilkS"))
-    (fp_line (start -4.65 -1.85) (end -1.6 -4.6)
+    (fp_line (start -4.185 -4.6) (end -4.185 4.6)
       (stroke (width 0.05) (type solid)) (layer "F.CrtYd"))
-    (fp_line (start -4.65 1.85) (end -4.65 -1.85)
+    (fp_line (start -4.185 4.6) (end 9.265 4.6)
       (stroke (width 0.05) (type solid)) (layer "F.CrtYd"))
-    (fp_line (start -1.6 -4.6) (end 11.85 -4.6)
+    (fp_line (start 9.265 -4.6) (end -4.185 -4.6)
       (stroke (width 0.05) (type solid)) (layer "F.CrtYd"))
-    (fp_line (start -1.6 4.6) (end -4.65 1.85)
+    (fp_line (start 9.265 4.6) (end 12.315 1.85)
       (stroke (width 0.05) (type solid)) (layer "F.CrtYd"))
-    (fp_line (start 11.85 -4.6) (end 11.85 4.6)
+    (fp_line (start 12.315 -1.85) (end 9.265 -4.6)
       (stroke (width 0.05) (type solid)) (layer "F.CrtYd"))
-    (fp_line (start 11.85 4.6) (end -1.6 4.6)
+    (fp_line (start 12.315 1.85) (end 12.315 -1.85)
       (stroke (width 0.05) (type solid)) (layer "F.CrtYd"))
-    (fp_line (start -4.15 -1.55) (end -4.15 1.55)
+    (fp_line (start -3.685 -4.05) (end 9.065 -4.05)
       (stroke (width 0.12) (type solid)) (layer "F.Fab"))
-    (fp_line (start -4.15 1.55) (end -1.4 4.05)
+    (fp_line (start -3.685 4.05) (end -3.685 -4.05)
       (stroke (width 0.12) (type solid)) (layer "F.Fab"))
-    (fp_line (start -1.4 -4.05) (end -4.15 -1.55)
+    (fp_line (start 9.065 -4.05) (end 11.815 -1.55)
       (stroke (width 0.12) (type solid)) (layer "F.Fab"))
-    (fp_line (start -1.4 4.05) (end 11.35 4.05)
+    (fp_line (start 9.065 4.05) (end -3.685 4.05)
       (stroke (width 0.12) (type solid)) (layer "F.Fab"))
-    (fp_line (start 11.35 -4.05) (end -1.4 -4.05)
+    (fp_line (start 11.815 -1.55) (end 11.815 1.55)
       (stroke (width 0.12) (type solid)) (layer "F.Fab"))
-    (fp_line (start 11.35 4.05) (end 11.35 -4.05)
+    (fp_line (start 11.815 1.55) (end 9.065 4.05)
       (stroke (width 0.12) (type solid)) (layer "F.Fab"))
     (pad "1" thru_hole roundrect (at 0 0) (size 6 6) (drill 4.5) (layers "*.Cu" "*.Mask") (roundrect_rratio 0.25)
@@
     (pts (xy 194.550002 144.750002) (xy 194.550002 83.74905))
     (height 16.379998)
-    (gr_text "61.0010 mm" (at 209.78 114.249526 90) (layer "Cmts.User")
+    (gr_text "2401.6123 mils" (at 209.78 114.249526 90) (layer "Cmts.User")
       (effects (font (size 1 1) (thickness 0.15)))
     )
@@
     (pts (xy 103.55 144.75) (xy 194.55 144.75))
     (height 7.36)
-    (gr_text "91.0000 mm" (at 149.05 150.96) (layer "Cmts.User")
+    (gr_text "3582.6772 mils" (at 149.05 150.96) (layer "Cmts.User")
       (effects (font (size 1 1) (thickness 0.15)))
     )
@@
     (pts (xy 194.54095 79.25) (xy 194.54095 149.260948))
     (height -10.94905)
-    (gr_text "70.0109 mm" (at 204.45 114.255474 90) (layer "Cmts.User")
+    (gr_text "2756.3365 mils" (at 204.45 114.255474 90) (layer "Cmts.User")
       (effects (font (size 1 1) (thickness 0.15)))
     )
@@
     (pts (xy 103.55 83.75) (xy 103.55 79.25))
     (height -6.95)
-    (gr_text "4.5000 mm" (at 96.557586 91.017586 90) (layer "Cmts.User")
+    (gr_text "177.1654 mils" (at 96.557586 91.017586 90) (layer "Cmts.User")
       (effects (font (size 1.5 1.5) (thickness 0.3)))
     )
@@
     (pts (xy 99.05 79.25) (xy 199.05 79.25))
     (height -6.68)
-    (gr_text "100.0000 mm" (at 149.05 70.77) (layer "Cmts.User")
+    (gr_text "3937.0079 mils" (at 149.05 70.77) (layer "Cmts.User")
       (effects (font (size 1.5 1.5) (thickness 0.3)))
     )
@@
     (pts (xy 103.55 83.75) (xy 99.05 83.75))
     (height 6.3)
-    (gr_text "4.5000 mm" (at 110.42 75.65) (layer "Cmts.User")
+    (gr_text "177.1654 mils" (at 110.42 75.65) (layer "Cmts.User")
       (effects (font (size 1.5 1.5) (thickness 0.3)))
     )
@@
         (xy 158.175 82.275)
         (xy 158.925 83.025)
-        (xy 158.925 83.025)
         (xy 160.475 84.575)
         (xy 163.475 84.575)
@@
         (xy 126.12 121.91)
         (xy 108.495 121.91)
-        (xy 108.495 121.91)
         (xy 101.645 121.91)
         (xy 101.27 122.285)
@@
         (xy 188.125 133.275)
         (xy 188.125 148.775)
-        (xy 143.95 148.775)
       )
     )
@@
         (xy 165.8 93.025)
         (xy 164.65 93.025)
-        (xy 164.65 93.025)
       )
     )
@@
         (xy 140.430414 96.444586)
         (xy 140.425 96.8)
-        (xy 140.425 96.8)
       )
