File: Hardware/Power_Supply.kicad_sch (KiCad schematic)
At the start: 20 parts, among them J2 Screw_Terminal_01x02, U11 B0505S, U3 XL1509-5.0, U9 LD1117

Commit message: Layout PCB
Parts:
- C14: value 470uF/35V -> 220uF/35V; footprint IVS_FOOTPRINTS:CP-Alu-SMD-10x10.5mm -> IVS_FOOTPRINTS:CP-Alu-SMD-8x10.5mm
Connections:
- net +24V: no longer C14.1, C15.1, U3.1 (VIN)
- net +24V_CS: now also C14.1, C15.1, U3.1 (VIN)
- net +5V: now also C24.1, U11.4 (Vout); no longer C16.1, C23.1, L2.1, R10.1, U11.2 (Vin)
- net +5V_CS: now also C16.1, C23.1, L2.1, R10.1, U11.2 (Vin), U3.3 (FB); no longer C24.1, U11.4 (Vout)
- net GND: now also C24.2, U11.3 (GNDout); no longer C14.2, C15.2, C16.2, C23.2, D1.1, LE3.2, U11.1 (GNDin), U3.4 (~{EN}), U3.5 (GND), U3.6 (GND), U3.7 (GND), U3.8 (GND)
- net GNDD: now also C14.2, C15.2, C16.2, C23.2, D1.1, LE3.2, U11.1 (GNDin), U3.4 (~{EN}), U3.5 (GND), U3.6 (GND), U3.7 (GND), U3.8 (GND); no longer C24.2, U11.3 (GNDout)
- net at D1.2, L2.2, U3.2 (OUT): no longer U3.3 (FB)
Other:
- moved on the sheet: F1, J2

Commit message: Update components
Parts:
- C14, C16: symbol Device:C -> Device:C_Polarized
- C23: footprint Capacitor_SMD:CP_Elec_4x5.4 -> IVS_FOOTPRINTS:C_1206; symbol Device:C -> Device:C_Polarized
- C24: value 10uF/16V -> 10uF/10V; footprint Capacitor_SMD:CP_Elec_4x5.4 -> IVS_FOOTPRINTS:C_1206; symbol Device:C -> Device:C_Polarized
- L2: footprint Inductor_SMD:L_1812_4532Metric -> Inductor_SMD:L_7.3x7.3_H4.5
Changed lines of the file:
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@@
       (effects (font (size 1.27 1.27)))
     )
-    (property "Footprint" "Inductor_SMD:L_1812_4532Metric" (at 114.935 132.715 0)
+    (property "Footprint" "Inductor_SMD:L_7.3x7.3_H4.5" (at 114.935 132.715 0)
       (effects (font (size 1.27 1.27)) hide)
     )
@@
     )
   )
-  (symbol (lib_id "Device:C") (at 60.325 137.795 0) (unit 1)
+  (symbol (lib_id "Device:C_Polarized") (at 60.325 137.795 0) (unit 1)
     (in_bom yes) (on_board yes) (dnp no)
     (property "Reference" "C14" (at 60.325 135.255 0)
@@
     )
   )
-  (symbol (lib_id "Device:C") (at 121.285 140.335 0) (unit 1)
+  (symbol (lib_id "Device:C_Polarized") (at 121.285 140.335 0) (unit 1)
     (in_bom yes) (on_board yes) (dnp no)
     (property "Reference" "C16" (at 121.285 137.795 0)
@@
     )
   )
-  (symbol (lib_id "Device:C") (at 60.96 95.25 0) (unit 1)
+  (symbol (lib_id "Device:C_Polarized") (at 60.96 95.25 0) (unit 1)
     (in_bom yes) (on_board yes) (dnp no)
     (property "Reference" "C23" (at 60.96 92.71 0)
@@
       (effects (font (size 1.27 1.27)) (justify left))
     )
-    (property "Footprint" "Capacitor_SMD:CP_Elec_4x5.4" (at 61.9252 99.06 0)
+    (property "Footprint" "IVS_FOOTPRINTS:C_1206" (at 61.9252 99.06 0)
       (effects (font (size 1.27 1.27)) hide)
     )
@@
     )
   )
-  (symbol (lib_id "Device:C") (at 97.155 95.25 0) (unit 1)
+  (symbol (lib_id "Device:C_Polarized") (at 97.155 95.25 0) (unit 1)
     (in_bom yes) (on_board yes) (dnp no)
     (property "Reference" "C24" (at 97.155 92.71 0)
       (effects (font (size 1.27 1.27)) (justify left))
     )
-    (property "Value" "10uF/16V" (at 97.155 97.79 0)
-      (effects (font (size 1.27 1.27)) (justify left))
-    )
-    (property "Footprint" "Capacitor_SMD:CP_Elec_4x5.4" (at 98.1202 99.06 0)
-      (effects (font (size 1.27 1.27)) hide)
-    )
+    (property "Value" "10uF/10V" (at 97.155 97.79 0)
+      (effects (font (size 1.27 1.27)) (justify left))
+    )
+    (property "Footprint" "IVS_FOOTPRINTS:C_1206" (at 98.1202 99.06 0)
+      (effects (font (size 1.27 1.27)) hide)
+    )

Commit message: Layout track part 2
Parts:
- added C11: 100nF, IVS_FOOTPRINTS:C_0603, symbol IVS_SYMBOLS:C
- added Q1: P_Mosfet, Package_TO_SOT_SMD:TO-252-2, symbol IVS_SYMBOLS:P_Mosfet_1G2D3S
- added R46: 100k, IVS_FOOTPRINTS:R_0603, symbol IVS_SYMBOLS:R
- added Z1: 15V, IVS_FOOTPRINTS:Package-Diode-D_MiniMELF, symbol IVS_SYMBOLS:D_Zener
- C15: footprint IVS_FOOTPRINTS:C_0603 -> IVS_FOOTPRINTS:C_1206
- R24: value 120R -> 1k
Connections:
- net +24V: now also Q1.2 (D); no longer F1.1
- net GND: no longer J2.2 (Pin_2)
- net GNDD: now also J2.2 (Pin_2), C11.2, R46.2
- new net: C11.1, Q1.1 (G), R46.1, Z1.1
- new net S: F1.1, Q1.3 (S), Z1.2
Other:
- moved on the sheet: F1

Commit message: Complete layout board
Connections:
- net XL1509_OUT: now reaches D1.2, L2.2, U3.2 (OUT)
Changed lines of the file:
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@@
   (junction (at 92.075 59.69) (diameter 0) (color 0 0 0 0)
   )
+  (junction (at 100.965 132.715) (diameter 0) (color 0 0 0 0)
+  )
   (junction (at 60.96 91.44) (diameter 0) (color 0 0 0 0)
   )
@@
     (stroke (width 0) (type default))
   )
+  (wire (pts (xy 100.965 125.73) (xy 100.965 132.715))
+    (stroke (width 0) (type default))
+  )
   (wire (pts (xy 121.285 151.765) (xy 107.315 151.765))
     (stroke (width 0) (type default))
@@
     (stroke (width 0) (type default))
   )
+  (wire (pts (xy 100.965 132.715) (xy 107.315 132.715))
+    (stroke (width 0) (type default))
+  )
   (wire (pts (xy 92.075 59.69) (xy 92.075 62.23))
     (stroke (width 0) (type default))
@@
     (stroke (width 0) (type default))
   )
-  (wire (pts (xy 99.695 132.715) (xy 107.315 132.715))
+  (wire (pts (xy 99.695 132.715) (xy 100.965 132.715))
     (stroke (width 0) (type default))
   )
@@
     (effects (font (size 1.27 1.27)) (justify left bottom))
   )
+  (label "XL1509_OUT" (at 100.965 125.73 0) (fields_autoplaced)
+    (effects (font (size 1.27 1.27)) (justify left bottom))
+  )

Commit message: Update README
Parts:
- removed C23: 4.7uF/16V, IVS_FOOTPRINTS:C_1206, symbol Device:C_Polarized
- removed C24: 10uF/10V, IVS_FOOTPRINTS:C_1206, symbol Device:C_Polarized
- added C10: 10uF/16V, IVS_FOOTPRINTS:C_0603, symbol IVS_SYMBOLS:C
- added C10: 4.7uF/25V, IVS_FOOTPRINTS:C_0603, symbol IVS_SYMBOLS:C
- added F3: 30V/3A, Fuse:Fuse_Bourns_MF-RG300, symbol IVS_SYMBOLS:Fuse
- added J2: Screw_Terminal_01x02, IVS_FOOTPRINTS:Conn-Vert-THT-2P-7.20mm-XT60_F, symbol Connector:Screw_Terminal_01x02
- Q1: value P_Mosfet -> IRF4905STRLPBF
Connections:
- net +24V_CS: now also F3.2
- net +5V: now also C10.1
- net +5V_CS: now also C10.1
- net GND: now also C10.2
- net GNDD: now also C10.2, J2.2 (Pin_2)
- new net: F3.1, J2.1 (Pin_1)
Other:
- note added: "Output JY01"
- moved on the sheet: Q1
