File: Hardware/STM32F103.kicad_sch (KiCad schematic)
At the start: 21 parts, among them J3 Conn_02x04_Counter_Clockwise, SW3 SW_Push, U5 MCU_STM32F103C8Tx, Y1 8Mhz

Commit message: Fix bug schematic
Parts:
- removed J3: Conn_02x04_Counter_Clockwise, Connector_IDC:IDC-Header_2x04_P2.54mm_Vertical, symbol Connector_Generic:Conn_02x04_Counter_Clockwise
- added J12: Conn_01x04_Male, Connector_PinHeader_2.54mm:PinHeader_1x04_P2.54mm_Vertical, symbol IVS_SYMBOLS:Conn_01x04_Male
- added J8: Conn_02x04_Odd_Even, Connector_IDC:IDC-Header_2x04_P2.54mm_Vertical, symbol Connector_Generic:Conn_02x04_Odd_Even
- added J9: Conn_01x07_Pin, Connector_PinHeader_2.54mm:PinHeader_1x07_P2.54mm_Vertical, symbol Connector:Conn_01x07_Pin
Connections:
- net +3V3_MCU: now also J8.7 (Pin_7)
- net +5VA: now also J8.8 (Pin_8)
- net GND: now also J8.5 (Pin_5), J8.6 (Pin_6)
- net RX_LOG: now also J8.2 (Pin_2)
- net SWCLK: now also J8.1 (Pin_1)
- net SWDIO: now also J8.3 (Pin_3)
- net TX_LOG: now also J8.4 (Pin_4)
- net PA5: now reaches U5.15 (PA5/SPI1_SCK/ADC12_IN5)
- net PB0: now reaches U5.18 (PB0/ADC12_IN8/TIM3_CH3/TIM1_CH2N)
- net PB0: now also J9.1 (Pin_1)
- net PB1: now reaches U5.19 (PB1/ADC12_IN9/TIM3_CH4/TIM1_CH3N)
- net PB1: now also J9.2 (Pin_2)
- net PB14: now reaches U5.27 (PB14/SPI2_MISO/USART3_RTS/TIM1_CH2N)
- net PB14: now also J9.6 (Pin_6)
- net PB15: now reaches U5.28 (PB15/SPI2_MOSI/TIM1_CH3N)
- net PB15: now also J9.7 (Pin_7)
- net PA8: now reaches U5.29 (PA8/USART1_CK/TIM1_CH1/MCO)
- net PA8: now also J12.1 (Pin_1)
- net PA9: now reaches U5.30 (PA9/USART1_TX/TIM1_CH2)
- net PA9: now also J12.2 (Pin_2)
- net PA10: now reaches U5.31 (PA10/USART1_RX/TIM1_CH3)
- net PA10: now also J12.3 (Pin_3)
- net PA15: now reaches U5.38 (PA15/JTDI)
- net PA15: now also J12.4 (Pin_4)
- net PB3: now reaches U5.39 (PB3/JTDO/TIM2_CH2/TRACESWO/SPI1_SCK)
- net PB3: now also J9.3 (Pin_3)
- net PB4: now reaches U5.40 (PB4/JNTRST/TIM3_CH1/SPI1_MISO)
- net PB4: now also J9.4 (Pin_4)
- net PB5: now reaches U5.41 (PB5/TIM3_CH2/SPI1_MOSI/I2C1_SMBAI)
- net PB5: now also J9.5 (Pin_5)

Commit message: Layout track part 2
Parts:
- J12: footprint Connector_PinHeader_2.54mm:PinHeader_1x04_P2.54mm_Vertical -> IVS_FOOTPRINTS:Conn-Horz-SMD-4P-2.54mm-PinHeader
- J9: footprint Connector_PinHeader_2.54mm:PinHeader_1x07_P2.54mm_Vertical -> IVS_FOOTPRINTS:Conn-Horz-SMD-7P-2.54mm-PinHeader
Changed lines of the file:
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@@
 (kicad_sch (version 20230121) (generator eeschema)
   (paper "A4")
-  (bus_alias "CAN" (members "CANH" "CANL"))
-  (bus_alias "I2C" (members "SCL" "SDA"))
   (bus_alias "DC_MOTOR" (members "PWM_L1" "PWM_R1" "PWM_L2" "PWM_R2"))
   (bus_alias "SPI" (members "MISO" "MOSI" "SCK" "CS"))
   (bus_alias "En" (members "EnA_1" "EnB_1" "EnA_2" "EnB_2"))
+  (bus_alias "CAN" (members "CANH" "CANL"))
+  (bus_alias "I2C" (members "SCL" "SDA"))
   (junction (at 212.09 124.46) (diameter 0) (color 0 0 0 0)
   )
@@
       (effects (font (size 1.27 1.27)))
     )
-    (property "Footprint" "Connector_PinHeader_2.54mm:PinHeader_1x04_P2.54mm_Vertical" (at 32.385 179.07 0)
+    (property "Footprint" "IVS_FOOTPRINTS:Conn-Horz-SMD-4P-2.54mm-PinHeader" (at 32.385 179.07 0)
       (effects (font (size 1.27 1.27)) hide)
     )
@@
       (effects (font (size 1.27 1.27)))
     )
-    (property "Footprint" "Connector_PinHeader_2.54mm:PinHeader_1x07_P2.54mm_Vertical" (at 32.385 162.56 0)
-      (effects (font (size 1.27 1.27)) hide)
-    )
+    (property "Footprint" "IVS_FOOTPRINTS:Conn-Horz-SMD-7P-2.54mm-PinHeader" (at 32.385 162.56 0)
+      (effects (font (size 1.27 1.27)) hide)
+    )

Commit message: Complete layout board
Connections:
- net PB0: now also J9.6 (Pin_6); no longer J9.1 (Pin_1)
- net PB1: now also J9.7 (Pin_7); no longer J9.2 (Pin_2)
- net PB14: now also J9.5 (Pin_5); no longer J9.6 (Pin_6)
- net PB15: now also J9.4 (Pin_4); no longer J9.7 (Pin_7)
- net PB4: now also J9.2 (Pin_2); no longer J9.4 (Pin_4)
- net PB5: now also J9.1 (Pin_1); no longer J9.5 (Pin_5)
- net PC13: now reaches R14.2, U5.2 (PC13/TAMPER-RTC)
Changed lines of the file:
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@@
 (kicad_sch (version 20230121) (generator eeschema)
   (paper "A4")
-  (bus_alias "DC_MOTOR" (members "PWM_L1" "PWM_R1" "PWM_L2" "PWM_R2"))
   (bus_alias "SPI" (members "MISO" "MOSI" "SCK" "CS"))
   (bus_alias "En" (members "EnA_1" "EnB_1" "EnA_2" "EnB_2"))
   (bus_alias "CAN" (members "CANH" "CANL"))
+  (bus_alias "DC_MOTOR" (members "PWM_L1" "PWM_R1" "PWM_L2" "PWM_R2"))
   (bus_alias "I2C" (members "SCL" "SDA"))
   (junction (at 212.09 124.46) (diameter 0) (color 0 0 0 0)
@@
   (junction (at 33.02 95.885) (diameter 0) (color 0 0 0 0)
   )
+  (junction (at 55.245 74.295) (diameter 0) (color 0 0 0 0)
+  )
   (junction (at 108.585 130.175) (diameter 0) (color 0 0 0 0)
   )
@@
     (stroke (width 0) (type default))
   )
+  (wire (pts (xy 55.245 74.295) (xy 57.785 74.295))
+    (stroke (width 0) (type default))
+  )
   (wire (pts (xy 256.54 102.87) (xy 264.16 102.87))
     (stroke (width 0) (type default))
@@
     (stroke (width 0) (type default))
   )
+  (wire (pts (xy 55.245 71.755) (xy 55.245 74.295))
+    (stroke (width 0) (type default))
+  )
   (wire (pts (xy 236.855 27.94) (xy 244.475 27.94))
     (stroke (width 0) (type default))
@@
     (stroke (width 0) (type default))
   )
-  (wire (pts (xy 53.975 74.295) (xy 57.785 74.295))
+  (wire (pts (xy 53.975 74.295) (xy 55.245 74.295))
     (stroke (width 0) (type default))
   )
@@
     (effects (font (size 1.27 1.27)) (justify left bottom))
   )
-  (label "PB5" (at 44.45 165.1 0) (fields_autoplaced)
+  (label "PB5" (at 44.45 154.94 0) (fields_autoplaced)
     (effects (font (size 1.27 1.27)) (justify left bottom))
   )
@@
     (effects (font (size 1.27 1.27)) (justify left bottom))
   )
-  (label "PB0" (at 44.45 154.94 0) (fields_autoplaced)
+  (label "PB0" (at 44.45 167.64 0) (fields_autoplaced)
     (effects (font (size 1.27 1.27)) (justify left bottom))
   )
@@
     (effects (font (size 1.27 1.27)) (justify left bottom))
   )
-  (label "PB4" (at 44.45 162.56 0) (fields_autoplaced)
+  (label "PB4" (at 44.45 157.48 0) (fields_autoplaced)
     (effects (font (size 1.27 1.27)) (justify left bottom))
   )
@@
     (effects (font (size 1.27 1.27)) (justify left bottom))
   )
-  (label "PB14" (at 44.45 167.64 0) (fields_autoplaced)
+  (label "PB14" (at 44.45 165.1 0) (fields_autoplaced)
     (effects (font (size 1.27 1.27)) (justify left bottom))
   )
@@
     (effects (font (size 1.27 1.27)) (justify left bottom))
   )
-  (label "PB15" (at 44.45 170.18 0) (fields_autoplaced)
+  (label "PB15" (at 44.45 162.56 0) (fields_autoplaced)
     (effects (font (size 1.27 1.27)) (justify left bottom))
   )
@@
     (effects (font (size 1.27 1.27)) (justify left bottom))
   )
-  (label "PB1" (at 44.45 157.48 0) (fields_autoplaced)
+  (label "PB1" (at 44.45 170.18 0) (fields_autoplaced)
     (effects (font (size 1.27 1.27)) (justify left bottom))
   )
@@
     (effects (font (size 1.27 1.27)) (justify right bottom))
   )
+  (label "PC13" (at 55.245 71.755 0) (fields_autoplaced)
+    (effects (font (size 1.27 1.27)) (justify left bottom))
+  )
   (label "OSC_IN" (at 252.095 48.26 0) (fields_autoplaced)

Commit message: Update README
Connections:
- net PB15 renamed MCU.PWM_EN
Changed lines of the file:
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@@
 (kicad_sch (version 20230121) (generator eeschema)
   (paper "A4")
+  (bus_alias "I2C" (members "SCL" "SDA"))
   (bus_alias "SPI" (members "MISO" "MOSI" "SCK" "CS"))
+  (bus_alias "DC_MOTOR" (members "PWM_L1" "PWM_R1" "PWM_L2" "PWM_R2"))
+  (bus_alias "CAN" (members "CANH" "CANL"))
   (bus_alias "En" (members "EnA_1" "EnB_1" "EnA_2" "EnB_2"))
-  (bus_alias "CAN" (members "CANH" "CANL"))
-  (bus_alias "DC_MOTOR" (members "PWM_L1" "PWM_R1" "PWM_L2" "PWM_R2"))
-  (bus_alias "I2C" (members "SCL" "SDA"))
   (junction (at 212.09 124.46) (diameter 0) (color 0 0 0 0)
   )
@@
     (stroke (width 0) (type default))
   )
+  (wire (pts (xy 49.53 122.555) (xy 57.785 122.555))
+    (stroke (width 0) (type default))
+  )
   (bus (pts (xy 266.7 95.25) (xy 266.7 97.79))
     (stroke (width 0) (type default))
@@
     (stroke (width 0) (type default))
   )
-  (wire (pts (xy 50.8 122.555) (xy 57.785 122.555))
-    (stroke (width 0) (type default))
-  )
   (wire (pts (xy 219.71 98.425) (xy 222.885 98.425))
     (stroke (width 0) (type default))
@@
   )
   (wire (pts (xy 113.665 130.175) (xy 113.665 131.445))
+    (stroke (width 0) (type default))
+  )
+  (wire (pts (xy 49.53 121.92) (xy 49.53 122.555))
     (stroke (width 0) (type default))
   )
@@
     (effects (font (size 1.27 1.27)) (justify left bottom))
   )
-  (label "PB15" (at 50.8 122.555 0) (fields_autoplaced)
-    (effects (font (size 1.27 1.27)) (justify left bottom))
+  (label "MCU.PWM_EN" (at 49.53 121.92 180) (fields_autoplaced)
+    (effects (font (size 1.27 1.27)) (justify right bottom))
   )
   (label "PA9" (at 166.37 107.315 0) (fields_autoplaced)
